File: arduino_shield.brd (EAGLE design)
At the start: 91.4 x 53.3 mm, 22 parts, among them IC1 MPL3115A2LGA, U1 USD-SOCKETNEW, U2 74HC4050, U4 FGPMMOPA6H, X1 22-23-2021

Commit message: Updated design
Parts:
- removed COMMON, SW1, SW2, SW3, SW4: (no value), adafruit:1X01
- added S1, S2, S3, S4: TL1105SPF160Q, SparkFun-Switches:TACTILE_SWITCH_PTH_6.0MM
Connections:
- net GND: now also S1.1, S2.1, S3.1, S4.1; no longer COMMON.1
- net SW1: now also S1.3; no longer SW1.1
- net SW2: now also S2.3; no longer SW2.1
- net SW3: now also S3.3; no longer SW3.1
- net SW4: now also S4.3; no longer SW4.1
Routing:
- net SW3: track 34.1 -> 44.9 mm
- net SW4: track 20.1 -> 30.8 mm, vias 2 -> 1
- net SW1: track 63.7 -> 73.3 mm, vias 2 -> 3
- net SW2: track 47.0 -> 56.2 mm, vias 2 -> 3
- net SCL_5V: track 55.2 -> 59.1 mm, vias 0 -> 2
- net CS_5V: track 92.1 -> 92.9 mm, vias 4 -> 2
- net SDA_5V: vias 2 -> 0
