File: arduino_shield.sch (EAGLE design)
At the start: 22 parts, among them IC1 MPL3115A2LGA, U1 USD-SOCKETNEW, U2 74HC4050, U4 FGPMMOPA6H, X1 22-23-2021

Commit message: Updated design
Parts:
- removed COMMON, SW1, SW2, SW3, SW4: (no value), adafruit:PINHD-1X1
- added S1, S2, S3, S4: TL1105SPF160Q, SparkFun-Switches:MOMENTARY-SWITCH-SPST-PTH-6.0MM
Connections:
- net GND: now also S1.1, S2.1, S3.1, S4.1; no longer COMMON.1
- net SW1: now also S1.2; no longer SW1.1
- net SW2: now also S2.2; no longer SW2.1
- net SW3: now also S3.2; no longer SW3.1
- net SW4: now also S4.2; no longer SW4.1
Changed lines of the file:
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@@
 <?xml version="1.0" encoding="utf-8"?>
 <!DOCTYPE eagle SYSTEM "eagle.dtd">
-<eagle version="8.2.2">
+<eagle version="8.3.1">
 <drawing>
 <settings>
 <setting alwaysvectorfont="no"/>
+<setting keepoldvectorfont="yes"/>
 <setting verticaltext="up"/>
 </settings>
@@
 <part name="L1" library="wuerth-elektronik" deviceset="WE-CBF" device="_1206"/>
 <part name="LED1" library="adafruit" deviceset="LED" device="SMT1206"/>
-<part name="COMMON" library="adafruit" library_urn="urn:adsk.eagle:library:420" deviceset="PINHD-1X1" device=""/>
-<part name="SW1" library="adafruit" library_urn="urn:adsk.eagle:library:420" deviceset="PINHD-1X1" device=""/>
-<part name="SW2" library="adafruit" library_urn="urn:adsk.eagle:library:420" deviceset="PINHD-1X1" device=""/>
-<part name="SW3" library="adafruit" library_urn="urn:adsk.eagle:library:420" deviceset="PINHD-1X1" device=""/>
-<part name="SW4" library="adafruit" library_urn="urn:adsk.eagle:library:420" deviceset="PINHD-1X1" device=""/>
 <part name="GND13" library="supply" deviceset="GND_" device=""/>
+<part name="S1" library="SparkFun-Switches" deviceset="MOMENTARY-SWITCH-SPST" device="-PTH-6.0MM" value="TL1105SPF160Q"/>
+<part name="S2" library="SparkFun-Switches" deviceset="MOMENTARY-SWITCH-SPST" device="-PTH-6.0MM" value="TL1105SPF160Q"/>
+<part name="S3" library="SparkFun-Switches" deviceset="MOMENTARY-SWITCH-SPST" device="-PTH-6.0MM" value="TL1105SPF160Q"/>
+<part name="S4" library="SparkFun-Switches" deviceset="MOMENTARY-SWITCH-SPST" device="-PTH-6.0MM" value="TL1105SPF160Q"/>
 </parts>
 <sheets>
@@
 <wire x1="-20.32" y1="-63.5" x2="-20.32" y2="10.16" width="0.1524" layer="97" style="shortdash"/>
 <text x="-17.78" y="2.54" size="5.08" layer="97">GPS</text>
-<wire x1="-38.1" y1="40.64" x2="-111.76" y2="40.64" width="0.1524" layer="97" style="shortdash"/>
-<wire x1="-38.1" y1="17.78" x2="-111.76" y2="17.78" width="0.1524" layer="97" style="shortdash"/>
-<wire x1="-111.76" y1="17.78" x2="-111.76" y2="40.64" width="0.1524" layer="97" style="shortdash"/>
-<wire x1="-38.1" y1="17.78" x2="-38.1" y2="40.64" width="0.1524" layer="97" style="shortdash"/>
-<text x="-109.22" y="33.02" size="5.08" layer="97">Buttons</text>
+<wire x1="-40.64" y1="66.04" x2="-83.82" y2="66.04" width="0.1524" layer="97" style="shortdash"/>
+<wire x1="-40.64" y1="20.32" x2="-83.82" y2="20.32" width="0.1524" layer="97" style="shortdash"/>
+<wire x1="-83.82" y1="20.32" x2="-83.82" y2="66.04" width="0.1524" layer="97" style="shortdash"/>
+<wire x1="-40.64" y1="20.32" x2="-40.64" y2="66.04" width="0.1524" layer="97" style="shortdash"/>
+<text x="-81.28" y="58.42" size="5.08" layer="97">Buttons</text>
 </plain>
 <instances>
@@
 <instance part="L1" gate="G$1" x="-2.54" y="-15.24"/>
 <instance part="LED1" gate="G$1" x="-2.54" y="-22.86" rot="R270"/>
-<instance part="COMMON" gate="G$1" x="-96.52" y="25.4"/>
-<instance part="SW1" gate="G$1" x="-81.28" y="25.4"/>
-<instance part="SW2" gate="G$1" x="-68.58" y="25.4"/>
-<instance part="SW3" gate="G$1" x="-55.88" y="25.4"/>
-<instance part="SW4" gate="G$1" x="-43.18" y="25.4"/>
-<instance part="GND13" gate="G$1" x="-106.68" y="20.32"/>
+<instance part="GND13" gate="G$1" x="-68.58" y="22.86"/>
+<instance part="S1" gate="G$1" x="-55.88" y="53.34"/>
+<instance part="S2" gate="G$1" x="-55.88" y="45.72"/>
+<instance part="S3" gate="G$1" x="-55.88" y="38.1"/>
+<instance part="S4" gate="G$1" x="-55.88" y="30.48"/>
 </instances>
 <busses>
@@
 </segment>
 <segment>
-<pinref part="COMMON" gate="G$1" pin="1"/>
-<pinref part="GND13" gate="G$1" pin="GND"/>
-<wire x1="-99.06" y1="25.4" x2="-106.68" y2="25.4" width="0.1524" layer="91"/>
-<wire x1="-106.68" y1="25.4" x2="-106.68" y2="22.86" width="0.1524" layer="91"/>
-<label x="-109.22" y="25.4" size="1.778" layer="95"/>
-</segment>
-<segment>
 <pinref part="B1" gate="G$1" pin="GND@0"/>
 <pinref part="GND6" gate="G$1" pin="GND"/>
 <wire x1="25.4" y1="30.48" x2="10.16" y2="30.48" width="0.1524" layer="91"/>
+</segment>
+<segment>
+<pinref part="S4" gate="G$1" pin="1"/>
+<wire x1="-60.96" y1="30.48" x2="-68.58" y2="30.48" width="0.1524" layer="91"/>
+<pinref part="S1" gate="G$1" pin="1"/>
+<wire x1="-60.96" y1="53.34" x2="-68.58" y2="53.34" width="0.1524" layer="91"/>
+<wire x1="-68.58" y1="30.48" x2="-68.58" y2="38.1" width="0.1524" layer="91"/>
+<wire x1="-68.58" y1="38.1" x2="-68.58" y2="45.72" width="0.1524" layer="91"/>
+<wire x1="-68.58" y1="45.72" x2="-68.58" y2="53.34" width="0.1524" layer="91"/>
+<wire x1="-68.58" y1="30.48" x2="-68.58" y2="25.4" width="0.1524" layer="91"/>
+<junction x="-68.58" y="30.48"/>
+<pinref part="GND13" gate="G$1" pin="GND"/>
+<label x="-68.58" y="33.02" size="1.778" layer="95"/>
+<pinref part="S3" gate="G$1" pin="1"/>
+<wire x1="-60.96" y1="38.1" x2="-68.58" y2="38.1" width="0.1524" layer="91"/>
+<junction x="-68.58" y="38.1"/>
+<pinref part="S2" gate="G$1" pin="1"/>
+<wire x1="-60.96" y1="45.72" x2="-68.58" y2="45.72" width="0.1524" layer="91"/>
+<junction x="-68.58" y="45.72"/>
 </segment>
 </net>
@@
 <net name="SW1" class="0">
 <segment>
-<wire x1="-83.82" y1="20.32" x2="-83.82" y2="25.4" width="0.1524" layer="91"/>
-<pinref part="SW1" gate="G$1" pin="1"/>
-<label x="-83.82" y="20.32" size="1.778" layer="95"/>
-</segment>
-<segment>
 <pinref part="B1" gate="G$1" pin="36"/>
 <wire x1="60.96" y1="63.5" x2="68.58" y2="63.5" width="0.1524" layer="91"/>
 <label x="63.5" y="63.5" size="1.778" layer="95"/>
 </segment>
+<segment>
+<pinref part="S1" gate="G$1" pin="2"/>
+<wire x1="-50.8" y1="53.34" x2="-45.72" y2="53.34" width="0.1524" layer="91"/>
+<label x="-48.26" y="53.34" size="1.778" layer="95"/>
+</segment>
 </net>
 <net name="SW2" class="0">
-<segment>
-<wire x1="-71.12" y1="20.32" x2="-71.12" y2="25.4" width="0.1524" layer="91"/>
-<pinref part="SW2" gate="G$1" pin="1"/>
-<label x="-71.12" y="20.32" size="1.778" layer="95"/>
-</segment>
 <segment>
 <pinref part="B1" gate="G$1" pin="38"/>
@@
 <label x="63.5" y="58.42" size="1.778" layer="95"/>
 </segment>
+<segment>
+<pinref part="S2" gate="G$1" pin="2"/>
+<wire x1="-50.8" y1="45.72" x2="-45.72" y2="45.72" width="0.1524" layer="91"/>
+<label x="-48.26" y="45.72" size="1.778" layer="95"/>
+</segment>
 </net>
 <net name="SW3" class="0">
-<segment>
-<wire x1="-58.42" y1="20.32" x2="-58.42" y2="25.4" width="0.1524" layer="91"/>
-<pinref part="SW3" gate="G$1" pin="1"/>
-<label x="-58.42" y="20.32" size="1.778" layer="95"/>
-</segment>
 <segment>
 <pinref part="B1" gate="G$1" pin="40"/>
@@
 <label x="63.5" y="53.34" size="1.778" layer="95"/>
 </segment>
+<segment>
+<pinref part="S3" gate="G$1" pin="2"/>
+<wire x1="-50.8" y1="38.1" x2="-45.72" y2="38.1" width="0.1524" layer="91"/>
+<label x="-48.26" y="38.1" size="1.778" layer="95"/>
+</segment>
 </net>
 <net name="SW4" class="0">
-<segment>
-<wire x1="-45.72" y1="20.32" x2="-45.72" y2="25.4" width="0.1524" layer="91"/>
-<pinref part="SW4" gate="G$1" pin="1"/>
-<label x="-45.72" y="20.32" size="1.778" layer="95"/>
-</segment>
 <segment>
 <pinref part="B1" gate="G$1" pin="42"/>
 <wire x1="60.96" y1="48.26" x2="68.58" y2="48.26" width="0.1524" layer="91"/>
 <label x="63.5" y="48.26" size="1.778" layer="95"/>
+</segment>
+<segment>
+<pinref part="S4" gate="G$1" pin="2"/>
+<wire x1="-50.8" y1="30.48" x2="-45.72" y2="30.48" width="0.1524" layer="91"/>
+<label x="-48.26" y="30.48" size="1.778" layer="95"/>
 </segment>
 </net>
@@
 <compatibility>
 <note version="8.2" severity="warning">
-Since Version 8.2, Eagle supports online libraries. The ids
+Since Version 8.2, EAGLE supports online libraries. The ids
 of those online libraries will not be understood (or retained)
 with this version.
